Commit message: temp

File: config/mowen_param/mowen.urdf (robot description, URDF)
Before this commit: robot mowen, 2 links, 1 joints
Links:
- link base_link: geometry collision mesh filename=package://robot_vs/config/mowen_param/meshes/base_link.STL; visual mesh filename=package://robot_vs/config/mowen_param/meshes/base_link.STL
